Commit message: conflict resolved

File: snake/robots/euclid_201709.gazebo.xacro (robot description, xacro)
@@ -8,3 +8,28 @@
   <xacro:include filename="$(find aerial_robot_simulation)/xacro/spinal.gazebo.xacro" />
   <xacro:gazebo_spinal robot_name="$(arg robot_name)" mag_frame="fc" />
+  <!-- gazebo plugin for docking mech -->
+  <gazebo>
+    <plugin name="gazebo_grasp_fix_1" filename="libgazebo_grasp_fix.so">
+      <arm>
+        <arm_name>docking_mech_1</arm_name>
+        <palm_link>dummy_palm_1</palm_link>
+        <gripper_link>dummy_gripper_1</gripper_link>
+	<arm_name>docking_mech_2</arm_name>
+        <palm_link>dummy_palm_2</palm_link>
+        <gripper_link>dummy_gripper_2</gripper_link>
+      </arm>
+      <arm>
+	<arm_name>docking_mech_2</arm_name>
+        <palm_link>dummy_palm_2</palm_link>
+        <gripper_link>dummy_gripper_2</gripper_link>
+      </arm>
+      <forces_angle_tolerance>90</forces_angle_tolerance>
+      <update_rate>50</update_rate>
+      <grip_count_threshold>0</grip_count_threshold>
+      <max_grip_count>1</max_grip_count>
+      <release_tolerance>1</release_tolerance>
+      <disable_collisions_on_attach>false</disable_collisions_on_attach>
+      <contact_topic>__default_topic__</contact_topic>
+    </plugin>
+  </gazebo>
 </robot>

File: snake/robots/euclid_201709.urdf.xacro (robot description, xacro)
@@ -6,3 +6,22 @@
   <xacro:include filename="$(find dragon)/robots/quad/euclid_201709.urdf.xacro" />
   <xacro:include filename="$(find snake)/urdf/snake_head.urdf.xacro" />
+  <link name="dummy_mouth">
+    <inertial>
+      <origin xyz="0 0 0" rpy="0 0 0"/>
+      <mass value="0.0001"/>
+      <inertia
+          ixx="0.0001"
+          iyy="0.0001"
+          izz="0.0001"
+          ixy="0.0"
+          ixz="0.0"
+          iyz="0.0"/>
+    </inertial>
+  </link>
+  <joint name="dummy_mouth_to_snake" type="fixed">
+    <parent link="snake"/>
+    <child link="dummy_mouth"/>
+    <origin rpy="0 0 0" xyz="0.20 0 0"/>
+    <axis xyz="1 0 0"/>
+  </joint>
 </robot>
